File: Alims.kicad_sch (KiCad schematic)
At the start: 17 parts, among them Q6 SUM110P06-08L, Q7 2N7002, Q8 2N7002

Commit message: CDR 2025 version WIP
Parts:
- removed C16, C19: 100nF, Capacitor_SMD:C_0603_1608Metric, symbol Device:C
- removed C17, C18: 470uF, Capacitor_THT:C_Radial_D8.0mm_H11.5mm_P3.50mm, symbol Device:C_Polarized_Small
- removed D6: ~, ComponentsEvo:DO-214AB, symbol Device:D_Small_Filled
- removed D7: 14.6V, Diode_SMD:D_SOD-323, symbol Device:D_Zener
- removed D8: LED, LED_SMD:LED_0603_1608Metric, symbol Device:LED
- removed Q6: SUM110P06-08L, Package_TO_SOT_SMD:TO-263-2, symbol Transistor_FET:QM6015D
- removed Q7, Q8: 2N7002, Package_TO_SOT_SMD:SOT-23, symbol Transistor_FET:2N7002
- removed R18, R21, R22, R23: 10k, Resistor_SMD:R_0603_1608Metric, symbol Device:R
- removed R19: 0, Resistor_SMD:R_0603_1608Metric, symbol Device:R
- removed R20: 4.7k, Resistor_SMD:R_0603_1608Metric, symbol Device:R
- removed R24: 0, Capacitor_SMD:C_0603_1608Metric, symbol Device:R
- added C12, C14, C4: 10uF, Capacitor_SMD:C_0603_1608Metric, symbol Device:C
- added C7: 430pF, Capacitor_SMD:C_0603_1608Metric, symbol Device:C
- added C9: 22uF, Capacitor_SMD:C_0603_1608Metric, symbol Device:C
- added D1, D9: D_Schottky, Diode_SMD:D_SOD-882, symbol Device:D_Schottky
- added R3, R5: 100k, Resistor_SMD:R_0603_1608Metric, symbol Device:R_Small
- added R4: 523k, Resistor_SMD:R_0603_1608Metric, symbol Device:R_Small
- added R7: 10k, Resistor_SMD:R_0603_1608Metric, symbol Device:R_Small
- added U6: TPS82130, Goldorak:MicroSiP, symbol Regulator_Switching:TPS82130
- added U7: AMS1117-3.3, Package_TO_SOT_SMD:SOT-89-3, symbol Regulator_Linear:AMS1117-3.3
Connections:
- net +3.3V: now also C14.1, U7.2 (VO)
- net GND: now also C12.2, C14.2, C4.2, U7.1 (GND)
- net GNDPWR: now also C7.2, C9.2, R5.1, R7.1, U6.3 (GND), U6.9 (GND)
- net VBAT_12V: now also C4.1, U6.2 (VIN)
- new net: R3.2, U6.7 (PG)
- new net: C7.1, U6.8 (SS/TR)
- new net: R4.1, R5.2, U6.6 (FB)
- new net +5VL: C12.1, D1.1 (K), D9.1 (K), R7.2, U6.1 (EN), U7.3 (VI)
- new net +5VP: C9.1, R3.1, R4.2, U6.4 (VOUT), U6.5 (VOUT)
- new net 5V_CAN: D1.2 (A)
- new net 5V_USB: D9.2 (A)
Other:
- note added: "3A max"
- note added: "Alim 3V3"
- note added: "Alim 5VL"
- note added: "Alim 5VP - LEDs Adressables"
- note added: "Res. pour Vout = 5V (calculé avec TI power designer)"
- note removed: "AU Status"
- note removed: "Commutation de l'alimentation PWR_12V via l'arrêt d'urgence"
- note removed: "PWR_12V"
- note removed: "Sheet I/O"
- company: Équipe Goldorak -> (none)
- title: Carte pneumatique -> (none)
