File: mcu.kicad_sch (KiCad schematic)
At the start: 17 parts, among them Q6 SUM110P06-08L, Q7 2N7002, Q8 2N7002

Commit message: CDR 2025 version WIP
Parts:
- removed C16, C19: 100nF, Capacitor_SMD:C_0603_1608Metric, symbol Device:C
- removed C17, C18: 470uF, Capacitor_THT:C_Radial_D8.0mm_H11.5mm_P3.50mm, symbol Device:C_Polarized_Small
- removed D6: ~, ComponentsEvo:DO-214AB, symbol Device:D_Small_Filled
- removed D7: 14.6V, Diode_SMD:D_SOD-323, symbol Device:D_Zener
- removed D8: LED, LED_SMD:LED_0603_1608Metric, symbol Device:LED
- removed Q6: SUM110P06-08L, Package_TO_SOT_SMD:TO-263-2, symbol Transistor_FET:QM6015D
- removed Q7, Q8: 2N7002, Package_TO_SOT_SMD:SOT-23, symbol Transistor_FET:2N7002
- removed R18, R21, R22, R23: 10k, Resistor_SMD:R_0603_1608Metric, symbol Device:R
- removed R19: 0, Resistor_SMD:R_0603_1608Metric, symbol Device:R
- removed R20: 4.7k, Resistor_SMD:R_0603_1608Metric, symbol Device:R
- removed R24: 0, Capacitor_SMD:C_0603_1608Metric, symbol Device:R
- added C29, C32: 10nF, Capacitor_SMD:C_0603_1608Metric, symbol Device:C
- added C30, C31: 100nF, Capacitor_SMD:C_0603_1608Metric, symbol Device:C
- added C5, C6: 18pF, Capacitor_SMD:C_0603_1608Metric, symbol Device:C
- added J13: STLINK, ConnectorsEvo:SAMTEC_FTSH-107-01-L-DV-K, symbol ConnectorsEvo:Conn_02x07_Odd_Even
- added R53, R54, R55, R56, R57, R58, R59, R60, R61, R62, R63, R64, R65, R66, R67, R68, R69, R70, R71, R72, R73, R74, R75, R76, R78, R79, R80, R81: 0, Resistor_SMD:R_0402_1005Metric, symbol Device:R
- added R77: 10k, Resistor_SMD:R_0402_1005Metric, symbol Device:R
- added SW1: 435431019840, ComponentsEvo:435431019840, symbol ComponentsEvo:435431019840
- added TP10, TP11, TP12, TP13, TP14, TP3, TP4, TP5, TP6, TP7, TP8: TestPoint_Small, TestPoint:TestPoint_Pad_D1.0mm, symbol Connector:TestPoint_Small
- added U5: STM32G474CEUx, Package_DFN_QFN:QFN-48-1EP_7x7mm_P0.5mm_EP5.6x5.6mm, symbol MCU_ST_STM32G4:STM32G474CEUx
- added Y1: 16 MHz, Crystal:Crystal_SMD_5032-4Pin_5.0x3.2mm, symbol Device:Crystal_GND24
Connections:
- net +3.3V: now also C29.1, C30.1, C31.1, C32.1, J13.3 (Pin_3), R77.2, U5.21 (VDDA), U5.23 (VDD), U5.35 (VDD), U5.48 (VDD)
- net GND: now also C29.2, C30.2, C31.2, C32.2, C5.1, C6.1, J13.11 (Pin_11), J13.5 (Pin_5), J13.7 (Pin_7), SW1.2, SW1.3, SW1.SH, U5.49 (VSS), Y1.2, Y1.4
- new net: R55.2, U5.26 (PB13)
- new net: TP14.1, U5.16 (PC4)
- new net: R63.1, U5.31 (PA9)
- new net: C5.2, U5.5 (PF0), Y1.1
- new net: R53.2, U5.45 (PB7)
- new net: R71.1, U5.8 (PA0)
- new net: TP3.1, U5.14 (PA6)
- new net: R54.2, U5.25 (PB12)
- new net: R66.2, U5.19 (PB2)
- new net: R78.1, U5.10 (PA2)
- new net: TP13.1, U5.39 (PC10)
- new net: R80.1, U5.12 (PA4)
- new net: R81.1, U5.11 (PA3)
- new net: C6.2, U5.6 (PF1), Y1.3
- new net: R76.2, U5.47 (PB9)
- new net: R61.1, U5.13 (PA5)
- new net: R70.2, U5.46 (PB8)
- new net: R59.1, U5.34 (PA12)
- new net: TP12.1, U5.29 (PC6)
- new net: R56.1, U5.38 (PA15)
- new net: R75.2, U5.22 (PB10)
- new net: R64.2, U5.17 (PB0)
- new net: TP7.1, U5.32 (PA10)
- new net: R67.2, U5.41 (PB3)
- new net: R57.1, U5.37 (PA14)
- new net: R79.2, U5.4 (PC15)
- new net: R73.2, U5.44 (PB6)
- new net: TP10.1, U5.40 (PC11)
- new net: R68.2, U5.42 (PB4)
- new net: TP8.1, U5.3 (PC14)
- new net: TP4.1, U5.15 (PA7)
- new net: R65.2, U5.18 (PB1)
- new net: TP11.1, U5.2 (PC13)
- new net: R74.2, U5.24 (PB11)
- new net: TP6.1, U5.27 (PB14)
- new net: TP5.1, U5.28 (PB15)
- new net: R62.1, U5.30 (PA8)
- new net: R60.1, U5.33 (PA11)
- new net: R58.1, U5.36 (PA13)
- new net: R69.2, U5.43 (PB5)
- new net: R72.1, U5.9 (PA1)
- new net BOOT0: R70.1
- new net CAN_RX: R54.1
- new net CAN_TX: R55.1
- new net DATA_LED: R61.2
- new net DS_COMP: R63.2
- new net DS_TURB: R62.2
- new net EV_1: R64.1
- new net EV_10: R74.1
- new net EV_11: R80.2
- new net EV_2: R65.1
- new net EV_3: R66.1
- new net EV_4: R79.1
- new net EV_5: R68.1
- new net EV_6: R69.1
- new net EV_7: R73.1
- new net EV_8: R76.1
- new net EV_9: R75.1
- new net EV_P: R72.2
- new net NRST: J13.12 (Pin_12), R77.1, SW1.1, SW1.4, U5.7 (PG10)
- new net SCL: R56.2
- new net SDA: R53.1
- new net SWDIO: J13.4 (Pin_4), R58.2
- new net SWO: J13.8 (Pin_8), R67.1
- new net SWTCK: J13.6 (Pin_6), R57.2
- new net USB_DN: R60.2
- new net USB_DP: R59.2
- new net VAC: R71.2
- new net VCP_RX: J13.13 (Pin_13), R81.2
- new net VCP_TX: J13.14 (Pin_14), R78.2
- no-connect marks 0 -> 6
Other:
- note removed: "AU Status"
- note removed: "Commutation de l'alimentation PWR_12V via l'arrêt d'urgence"
- note removed: "PWR_12V"
- note removed: "Sheet I/O"
- company: Équipe Goldorak -> (none)
- title: Carte pneumatique -> (none)
