File: 12v-actuators-pcb.kicad_pcb (KiCad board)
At the start: 2 copper layers, 245.9 x 197.5 mm, 206 parts, among them J1 690367280876, J10 ESC_35_1_P, J11 690367280876, J12 ESC_35_2_S, J13 Alim Pompe, J14 690367280876, J15 BOOT0, J16 690367280876, J17 690367280876, J18 690367280876, J19 Alim EV, J2 3.5mm WR-TBL, J20 Alim EV, J21 Alim EV, J22 Alim EV, J23 Alim EV, J24 Alim EV, J25 Alim EV, J26 Alim EV, J27 Alim EV, J28 Alim EV, J29 Alim EV, J3 690367280676, J30 Alim EV, J4 STLINK, J5 USB_B_Mini, J6 ESC_35_1_P, J7 RGBA_LEDs, J8 CAN, J9 ESC_35_1_S, Q1 G2302, Q10 G2302, Q11 G2302, Q12 G2302, Q13 G2302, Q14 G2302, Q15 G2302, Q16 G2302, Q17 G2302, Q18 G2302, Q2 G2302, Q3 G2302, Q4 G2302, Q5 G2302, Q6 SUM110P06-08L, Q7 2N7002, Q8 2N7002, SW1 435431019840, U1 MCP2551-I-SN, U2 TCA9517DR, U3 WSEN-PDUS, U4 STM32G474CEUx, U5 AMS1117-3.3, U6 TPS82130, Y1 16 MHz

Commit message: ajout regle routage JLCPCB, fin placement grossier et debut reassignation. ajout de led temoin, homogeinisation empreinte passif et remplacement 0ohm par empreintre jumper PCB 0402.
Parts:
- removed R32, R35, R54, R55, R56, R57, R59, R60, R61, R62, R63, R65, R66, R67, R68, R69, R70, R71, R72, R73, R74, R77, R83, R84, R85: 0, Resistor_SMD:R_0402_1005Metric
- added D11: LED, LED_SMD:LED_0603_1608Metric, F.Cu at (222.0, 59.0)
- added D20: LED, LED_SMD:LED_0603_1608Metric, F.Cu at (199.5, 74.5)
- added D21: LED, LED_SMD:LED_0603_1608Metric, F.Cu at (175.5, 66.5)
- added JP1: SolderJumper_2_Bridged, 12V-actuators_pcb:R_0402_1005Metric_jumperClosed, F.Cu at (206.5, 56.5)
- added JP10: SolderJumper_2_Bridged, 12V-actuators_pcb:R_0402_1005Metric_jumperClosed, F.Cu at (177.0, 56.5)
- added JP11: SolderJumper_2_Bridged, 12V-actuators_pcb:R_0402_1005Metric_jumperClosed, F.Cu at (178.0, 56.5)
- added JP12: SolderJumper_2_Bridged, 12V-actuators_pcb:R_0402_1005Metric_jumperClosed, F.Cu at (180.5, 90.5)
- added JP13: SolderJumper_2_Bridged, 12V-actuators_pcb:R_0402_1005Metric_jumperClosed, F.Cu at (182.5, 90.5)
- added JP14: SolderJumper_2_Bridged, 12V-actuators_pcb:R_0402_1005Metric_jumperClosed, F.Cu at (194.5, 84.0)
- added JP15: SolderJumper_2_Bridged, 12V-actuators_pcb:R_0402_1005Metric_jumperClosed, F.Cu at (193.5, 61.5)
- added JP16: SolderJumper_2_Bridged, 12V-actuators_pcb:R_0402_1005Metric_jumperClosed, F.Cu at (180.5, 71.5)
- added JP17: SolderJumper_2_Bridged, 12V-actuators_pcb:R_0402_1005Metric_jumperClosed, F.Cu at (193.5, 73.0)
- added JP18: SolderJumper_2_Bridged, 12V-actuators_pcb:R_0402_1005Metric_jumperClosed, F.Cu at (194.5, 73.0)
- added JP19: SolderJumper_2_Bridged, 12V-actuators_pcb:R_0402_1005Metric_jumperClosed, F.Cu at (179.0, 56.5)
- added JP2: SolderJumper_2_Bridged, 12V-actuators_pcb:R_0402_1005Metric_jumperClosed, F.Cu at (203.5, 56.5)
- added JP20: SolderJumper_2_Bridged, 12V-actuators_pcb:R_0402_1005Metric_jumperClosed, F.Cu at (196.5, 73.0)
- added JP21: SolderJumper_2_Bridged, 12V-actuators_pcb:R_0402_1005Metric_jumperClosed, F.Cu at (207.5, 56.5)
- added JP22: SolderJumper_2_Bridged, 12V-actuators_pcb:R_0402_1005Metric_jumperClosed, F.Cu at (193.5, 58.5)
- added JP23: SolderJumper_2_Bridged, 12V-actuators_pcb:R_0402_1005Metric_jumperClosed, F.Cu at (193.5, 59.5)
- added JP24: SolderJumper_2_Bridged, 12V-actuators_pcb:R_0402_1005Metric_jumperClosed, F.Cu at (193.5, 60.5)
- added JP25: SolderJumper_2_Bridged, 12V-actuators_pcb:R_0402_1005Metric_jumperClosed, F.Cu at (195.5, 73.0)
- added JP26: SolderJumper_2_Bridged, 12V-actuators_pcb:R_0402_1005Metric_jumperClosed, F.Cu at (175.0, 69.0)
- added JP27: SolderJumper_2_Bridged, 12V-actuators_pcb:R_0402_1005Metric_jumperClosed, F.Cu at (175.0, 71.0)
- added JP28: SolderJumper_2_Bridged, 12V-actuators_pcb:R_0402_1005Metric_jumperClosed, F.Cu at (192.5, 84.0)
- added JP3: SolderJumper_2_Bridged, 12V-actuators_pcb:R_0402_1005Metric_jumperClosed, F.Cu at (204.5, 56.5)
- added JP4: SolderJumper_2_Bridged, 12V-actuators_pcb:R_0402_1005Metric_jumperClosed, F.Cu at (205.5, 56.5)
- added JP5: SolderJumper_2_Bridged, 12V-actuators_pcb:R_0402_1005Metric_jumperClosed, F.Cu at (190.0, 56.0)
- added JP6: SolderJumper_2_Bridged, 12V-actuators_pcb:R_0402_1005Metric_jumperClosed, F.Cu at (191.0, 56.0)
- added JP7: SolderJumper_2_Bridged, 12V-actuators_pcb:R_0402_1005Metric_jumperClosed, F.Cu at (192.5, 56.0)
- added JP8: SolderJumper_2_Bridged, 12V-actuators_pcb:R_0402_1005Metric_jumperClosed, F.Cu at (193.5, 84.0)
- added JP9: SolderJumper_2_Bridged, 12V-actuators_pcb:R_0402_1005Metric_jumperClosed, F.Cu at (193.5, 56.0)
- added TP8: TestPoint_Small, TestPoint:TestPoint_Pad_D1.0mm, F.Cu at (188.5, 71.0)
- C29, C30, C4: footprint Capacitor_SMD:C_0603_1608Metric -> Capacitor_SMD:C_0805_2012Metric
- R19, R86: footprint Resistor_SMD:R_0402_1005Metric -> 12V-actuators_pcb:R_0402_1005Metric_jumperClosed
- R29: value 0 -> 10k; footprint Resistor_SMD:R_0402_1005Metric -> Resistor_SMD:R_0603_1608Metric
- R30: value 0 -> 4.7k; footprint Resistor_SMD:R_0402_1005Metric -> Resistor_SMD:R_0603_1608Metric
- R31: value 0 -> 1k; footprint Resistor_SMD:R_0402_1005Metric -> Resistor_SMD:R_0603_1608Metric
- R81: footprint Resistor_SMD:R_0402_1005Metric -> Resistor_SMD:R_0603_1608Metric
- moved H8 183.7 mm to (-10.5, -5.60), turned to -90 degrees
- moved H9 183.7 mm to (178.0, -5.60), turned to -90 degrees
- moved R39 178.6 mm to (170.5, -8.00), turned to -90 degrees
- moved R43 178.3 mm to (168.0, -10.0), turned to 180 degrees
- moved R47 177.8 mm to (0.00, -10.0), turned to 180 degrees
- moved Q12 175.1 mm to (168.0, -7.00), turned to -90 degrees
- moved Q15 174.6 mm to (0.00, -7.00), turned to -90 degrees
- moved R36 173.3 mm to (2.50, -8.00), turned to -90 degrees
- moved R40 173.3 mm to (165.0, -8.00), turned to -90 degrees
- moved R44 173.2 mm to (162.5, -10.0), turned to 180 degrees
- moved R46 171.8 mm to (6.50, -10.0), turned to 180 degrees
- moved D15 171.5 mm to (168.0, -3.50), turned to 0 degrees
- moved D12 171.0 mm to (0.00, -3.50), turned to 180 degrees
- moved Q13 169.9 mm to (162.5, -7.00), turned to -90 degrees
- moved Q10 168.5 mm to (6.50, -7.00), turned to -90 degrees
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Connections:
- net Net-(U4-PC10) renamed /MCU et capteurs/TP3
- net Net-(U4-PC11) renamed /MCU et capteurs/TP4
- net Net-(U4-PC13) renamed /MCU et capteurs/TP5
- net Net-(U4-PC14) renamed /MCU et capteurs/TP6
- net Net-(U4-PC4) renamed /MCU et capteurs/TP1
- net Net-(U4-PC6) renamed /MCU et capteurs/TP2
- net Net-(U4-PF0) renamed /MCU et capteurs/OSC0
- net Net-(U4-PF1) renamed /MCU et capteurs/OSC1
- J15 pad 1: /MCU et capteurs/BOOT0 -> /MCU et capteurs/SCL
- R29 pad 1: /EV_4 -> Net-(D11-K)
- R29 pad 2: Net-(U4-PC15) -> Net-(J6-Pin_2)
- R30 pad 1: /EV_1 -> Net-(D20-K)
- R30 pad 2: Net-(U4-PB0) -> GNDPWR
- R31 pad 1: /EV_2 -> Net-(D21-K)
- R31 pad 2: Net-(U4-PB1) -> GND
- TP7 pad 1: Net-(U4-PB14) -> /MCU et capteurs/VREF_uC
- U4 pad 1: unconnected-(U4-VBAT-Pad1) -> /MCU et capteurs/VBAT_uC
- U4 pad 10: Net-(U4-PA2) -> unconnected-(U4-PA2-Pad10)
- U4 pad 11: Net-(U4-PA3) -> unconnected-(U4-PA3-Pad11)
- U4 pad 12: Net-(U4-PA4) -> /MCU et capteurs/EV_11_J
- U4 pad 13: Net-(U4-PA5) -> /MCU et capteurs/DATA_LED_J
- U4 pad 14: Net-(U4-PA6) -> /MCU et capteurs/EV_P_J
- U4 pad 15: Net-(U4-PA7) -> /MCU et capteurs/VAC_J
- U4 pad 17: Net-(U4-PB0) -> /MCU et capteurs/EV_1_J
- U4 pad 18: Net-(U4-PB1) -> /MCU et capteurs/EV_2_J
- U4 pad 19: Net-(U4-PB2) -> /MCU et capteurs/EV_3_J
- U4 pad 20: unconnected-(U4-VREF+-Pad20) -> /MCU et capteurs/VREF_uC
- U4 pad 22: Net-(U4-PB10) -> /MCU et capteurs/EV_9_J
- U4 pad 24: Net-(U4-PB11) -> /MCU et capteurs/EV_10_J
- U4 pad 25: Net-(U4-PB12) -> unconnected-(U4-PB12-Pad25)
- U4 pad 26: Net-(U4-PB13) -> unconnected-(U4-PB13-Pad26)
- U4 pad 27: Net-(U4-PB14) -> /MCU et capteurs/LED_DBG
- U4 pad 28: Net-(U4-PB15) -> /MCU et capteurs/LED_EN_J
- U4 pad 30: Net-(U4-PA8) -> /MCU et capteurs/CAN_RX_J
- U4 pad 31: Net-(U4-PA9) -> /MCU et capteurs/VCP_TX_J
- U4 pad 32: Net-(U4-PA10) -> /MCU et capteurs/VCP_RX_J
- U4 pad 33: Net-(U4-PA11) -> /MCU et capteurs/USB_DN_J
- U4 pad 34: Net-(U4-PA12) -> /MCU et capteurs/USB_DP_J
- U4 pad 38: Net-(U4-PA15) -> /MCU et capteurs/CAN_TX_J
- U4 pad 4: Net-(U4-PC15) -> /MCU et capteurs/EV_4_J
- U4 pad 42: Net-(U4-PB4) -> /MCU et capteurs/EV_5_J
- U4 pad 43: Net-(U4-PB5) -> /MCU et capteurs/EV_6_J
- U4 pad 44: Net-(U4-PB6) -> /MCU et capteurs/EV_7_J
- U4 pad 45: Net-(U4-PB7) -> /MCU et capteurs/SDA_J
- U4 pad 46: /MCU et capteurs/BOOT0 -> /MCU et capteurs/SCL_J
- U4 pad 47: Net-(U4-PB9) -> /MCU et capteurs/EV_8_J
- U4 pad 8: Net-(U4-PA0) -> /MCU et capteurs/A_TEMP_J
- U4 pad 9: Net-(U4-PA1) -> /MCU et capteurs/A_PRES_J
Other:
- board size 245.9 x 197.5 mm -> 248.3 x 109.6 mm

Commit message: fin du placement et reassignation des pins uC
Parts:
- removed J15: BOOT0, Connector_PinHeader_2.54mm:PinHeader_1x02_P2.54mm_Vertical
- removed TP1, TP5, TP6, TP8: TestPoint_Small, TestPoint:TestPoint_Pad_D1.0mm
- added D22: LED, LED_SMD:LED_0603_1608Metric, F.Cu at (164.2, 59.0)
- added D23: LED, LED_SMD:LED_0603_1608Metric, F.Cu at (164.2, 62.2)
- added JP29: SolderJumper_2_Bridged, 12V-actuators_pcb:R_0402_1005Metric_jumperClosed, F.Cu at (181.5, 57.0)
- added R32: 1k, Resistor_SMD:R_0603_1608Metric, F.Cu at (168.2, 58.2)
- added R35: 1k, Resistor_SMD:R_0603_1608Metric, F.Cu at (168.2, 61.8)
- R24, R89: moved to B.Cu
- moved R24 71.1 mm to (168.0, 63.0), turned to -90 degrees
- moved TP2 48.8 mm to (191.5, 71.0)
- moved TP3 46.4 mm to (189.5, 69.0)
- moved TP4 46.4 mm to (191.5, 69.0)
- moved D21 15.6 mm to (164.2, 55.8)
- moved R89 13.6 mm to (225.0, 90.0), turned to -90 degrees
- moved R82 12.7 mm to (188.0, 73.0)
- moved R31 10.3 mm to (169.0, 55.5), turned to 0 degrees
- moved JP15 9.12 mm to (202.5, 60.0)
- moved JP10 8.06 mm to (178.0, 64.5), turned to 0 degrees
- moved JP2 7.02 mm to (196.5, 57.0)
- moved JP3 6.52 mm to (198.0, 57.0)
- moved C18 5.22 mm to (173.5, 57.5)
- moved JP16 5.15 mm to (178.0, 67.0), turned to 0 degrees
- moved JP25 5.10 mm to (196.5, 78.0)
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Connections:
- D21 pad 2: /MCU et capteurs/LED_DBG -> /MCU et capteurs/LED_DBG_1
- J11 pad 6: unconnected-(J11-Pad6) -> /EV_12
- R82 pad 1: Net-(J15-Pin_2) -> /MCU et capteurs/BOOT0
- U4 pad 1: /MCU et capteurs/VBAT_uC -> unconnected-(U4-VBAT-Pad1)
- U4 pad 10: unconnected-(U4-PA2-Pad10) -> /MCU et capteurs/DS_COMP_J
- U4 pad 11: unconnected-(U4-PA3-Pad11) -> /MCU et capteurs/DS_TURB_J
- U4 pad 12: /MCU et capteurs/EV_11_J -> /MCU et capteurs/VAC_J
- U4 pad 13: /MCU et capteurs/DATA_LED_J -> /MCU et capteurs/EV_P_J
- U4 pad 14: /MCU et capteurs/EV_P_J -> /MCU et capteurs/EV_4_J
- U4 pad 15: /MCU et capteurs/VAC_J -> /MCU et capteurs/EV_3_J
- U4 pad 16: /MCU et capteurs/TP1 -> /MCU et capteurs/EV_2_J
- U4 pad 18: /MCU et capteurs/EV_2_J -> /MCU et capteurs/EV_8_J
- U4 pad 19: /MCU et capteurs/EV_3_J -> /MCU et capteurs/EV_7_J
- U4 pad 2: /MCU et capteurs/TP5 -> /MCU et capteurs/TP2
- U4 pad 22: /MCU et capteurs/EV_9_J -> /MCU et capteurs/EV_6_J
- U4 pad 24: /MCU et capteurs/EV_10_J -> /MCU et capteurs/EV_5_J
- U4 pad 25: unconnected-(U4-PB12-Pad25) -> /MCU et capteurs/EV_12_J
- U4 pad 26: unconnected-(U4-PB13-Pad26) -> /MCU et capteurs/EV_11_J
- U4 pad 27: /MCU et capteurs/LED_DBG -> /MCU et capteurs/EV_10_J
- U4 pad 28: /MCU et capteurs/LED_EN_J -> /MCU et capteurs/EV_9_J
- U4 pad 29: /MCU et capteurs/TP2 -> /MCU et capteurs/LED_DBG_1
- U4 pad 3: /MCU et capteurs/TP6 -> /MCU et capteurs/TP3
- U4 pad 30: /MCU et capteurs/CAN_RX_J -> /MCU et capteurs/LED_DBG_2
- U4 pad 31: /MCU et capteurs/VCP_TX_J -> /MCU et capteurs/A_PRES_J
- U4 pad 32: /MCU et capteurs/VCP_RX_J -> /MCU et capteurs/LED_DBG_3
- U4 pad 38: /MCU et capteurs/CAN_TX_J -> /MCU et capteurs/SCL_J
- U4 pad 39: /MCU et capteurs/TP3 -> /MCU et capteurs/VCP_TX_J
- U4 pad 4: /MCU et capteurs/EV_4_J -> /MCU et capteurs/TP4
- U4 pad 40: /MCU et capteurs/TP4 -> /MCU et capteurs/VCP_RX_J
- U4 pad 42: /MCU et capteurs/EV_5_J -> /MCU et capteurs/LED_EN_J
- U4 pad 43: /MCU et capteurs/EV_6_J -> /MCU et capteurs/CAN_RX_J
- U4 pad 44: /MCU et capteurs/EV_7_J -> /MCU et capteurs/CAN_TX_J
- U4 pad 46: /MCU et capteurs/SCL_J -> /MCU et capteurs/BOOT0
- U4 pad 47: /MCU et capteurs/EV_8_J -> /MCU et capteurs/AU_STATUS_J
- U4 pad 8: /MCU et capteurs/A_TEMP_J -> /MCU et capteurs/DATA_LED_J
- U4 pad 9: /MCU et capteurs/A_PRES_J -> /MCU et capteurs/A_TEMP_J
